File: fw16_oculink8i.kicad_pcb (KiCad board)
At the start: 4 copper layers, 99.3 x 73.9 mm, 78 parts, among them J1 FXBeam, J2 x8 NPIO, J3 USB_A, J4 FAN_CON_L, J5 FAN_CON_R, SW1 SW_DPDT_x2, SW2 SW_DPDT_x2, U1 LM393, U2 BR24G32FVT-3GE2

Commit message: updated footprint for comparator for SOIC-8
JLCPCB has it as a standard component instead of extended, so 3 bucks cheaper (yay)
Parts:
- removed REF**: Symbol_ESD-Logo_CopperTop, Symbol:Symbol_ESD-Logo_CopperTop
- removed REF**: OSHW-Logo2_36.5x30mm_SilkScreen, Symbol:OSHW-Logo2_36.5x30mm_SilkScreen
- U1: footprint Package_SO:TSSOP-8_4.4x3mm_P0.65mm -> Package_SO:SOIC-8_3.9x4.9mm_P1.27mm
- moved R6 5.23 mm to (105.3, 40.2), turned to 0 degrees
- moved R8 3.76 mm to (105.3, 41.3), turned to 180 degrees
- moved R1 1.69 mm to (102.4, 40.3)
- moved R2 1.69 mm to (100.5, 40.3)
- moved C2 1.42 mm to (103.3, 41.2), turned to 180 degrees
- moved R5 0.42 mm to (96.7, 44.5)
- moved R7 0.40 mm to (97.8, 44.5)
Routing:
- net /CPRSNTB: track 27.0 -> 31.7 mm
- net Net-(U1B-+): track 2.70 -> 7.36 mm
- net /CLK_AUTO_EN1: track 6.54 -> 8.92 mm, vias 2 -> 0
- net /CLK_AUTO_EN2: track 7.05 -> 8.16 mm, vias 2 -> 0
- net GND: track 138.4 -> 139.5 mm
- net /CLKE_BIAS: track 9.68 -> 10.6 mm, vias 0 -> 5
