File: fw16_oculink8i.kicad_sch (KiCad schematic)
At the start: 55 parts, among them J1 Fan, J2 Fan, J3 FXBeam, J4 I2C, J5 USB_A, J6 x8 NPIO, SW1 SW_DPDT_x2, SW2 SW_DIP_x02, U1 BR24G32FVT-3GE2, U2 TL331LV, U3 TL331LV

Commit message: cleaned up the schematic and removed some redundant components
A big cleanup of the schematic so that it uses power signals instead of labels.

Some resistors where removed since they were redundant. Same with some caps and now only uses one type of switch.

The comparator is now a dual one that consumes a bit less power too.
Parts:
- removed C2, C3, C5: 0.1U, Capacitor_SMD:C_0402_1005Metric, symbol Device:C_Small
- removed J1, J2: Fan, FPC_Conn:AFC58-S04FIA_4Pin, symbol Connector_Generic:Conn_01x04
- removed R16, R17: 1K, Resistor_SMD:R_0402_1005Metric, symbol Device:R_Small
- removed R18, R20: 10K, Resistor_SMD:R_0402_1005Metric, symbol Device:R_Small
- removed R22, R23, R3, R30, R33, R34, R4, R5: 0R, Resistor_SMD:R_0402_1005Metric, symbol Device:R_Small
- removed R24, R25: 100K, Resistor_SMD:R_0402_1005Metric, symbol Device:R_Small
- removed R26, R27: 47K, Resistor_SMD:R_0402_1005Metric, symbol Device:R_Small
- removed SW2: SW_DIP_x02, Button_Switch_SMD:SW_DIP_SPSTx02_Slide_Copal_CHS-02B_W7.62mm_P1.27mm, symbol Switch:SW_DIP_x02
- removed U2, U3: TL331LV, Package_TO_SOT_SMD:SOT-23-5, symbol Comparator:TL331
- added J5: FAN_CON_R, FPC_Conn:AFC58-S04FIA_4Pin, symbol Connector_Generic_MountingPin:Conn_01x04_MountingPin
- added R1: 100K, Resistor_SMD:R_0402_1005Metric, symbol Device:R_Small
- added R2: 47K, Resistor_SMD:R_0402_1005Metric, symbol Device:R_Small
- added SW1, SW2: SW_DPDT_x2, Switches:SSSS820101, symbol Switch:SW_DPDT_x2
- added U1: LM393, Package_DIP:DIP-14_W7.62mm, symbol Comparator:LM393
- C1: value 0.1U -> 100n; now fitted
- C2: renamed from C4; value 0.1U -> 100n
- J4: value I2C -> FAN_CON_L; footprint Connector_JST:JST_SH_SM04B-SRSS-TB_1x04-1MP_P1.00mm_Horizontal -> FPC_Conn:AFC58-S04FIA_4Pin; now in the parts list
- R3: renamed from R9; value 4.7K -> 4k7
- R4: renamed from R6; value 4.7K -> 4k7
- renumbered J3 to J1, J6 to J2, J5 to J3, R14 to R10, R15 to R11, R7 to R14, R8 to R15, R11 to R16, R10 to R17, R19 to R18, R21 to R19, R36 to R20, R1 to R21, R28 to R5, R31 to R6, R29 to R7, R32 to R8, R2 to R9, SW1 to SW3, U1 to U2
Connections:
- net 3V3_CLK_EN1 is gone; now on net GND: C2.1
- net 3V3_CTRL is gone; now on net +3V3: J1.PA4 (3V3_ALW), J1.PB4 (3V3_ALW)
- net 3V3_ID is gone; now on net +3V3: J1.PA5 (3V3_ALW), J1.PB5 (3V3_ALW)
- net CLK_AUTO_EN1: now also SW1.6 (C), U1.1; no longer R18.1
- net CLK_AUTO_EN2: now also SW2.6 (C), U1.7; no longer R19.1
- net EEPROM_WP: now also R16.2; no longer R16.1
- net FAN0_PWM: now also J4.2 (Pin_2)
- net FAN0_SPD: now also J4.3 (Pin_3)
- net FAN1_PWM: now also J5.3 (Pin_3)
- net FAN1_SPD: now also J5.2 (Pin_2)
- net GND: now also C1.2, J3.5 (Shield), J4.4 (Pin_4), R21.2, R9.2, J5.4 (Pin_4), J5.MP (MountPin), R2.1, SW1.4 (A), SW2.4 (A), U1.4 (V-); no longer C1.1, C2.2, J4.1 (Pin_1), R21.1, R9.1
- net I2C_SCL: now also R3.2, U2.6 (SCL)
- net I2C_SDA: now also R4.1, U2.5 (SDA)
- net at J1.SL2 (ID1): now also R21.1; no longer R21.2
- net at R5.2, R7.1: now also U1.3 (+)
- net +3V3: now reaches R7.2
- net +3V3: now also C1.1, C2.2, R10.1, R12.1, R14.1, R16.1, R3.1, R4.2, R8.2, U2.8 (VCC), R1.1, U1.8 (V+)
- net at R6.2, R8.1: now also U1.5 (+)
- net at J1.PJ1 (ID0): now also R9.1; no longer R9.2
- net 12V_FAN renamed +12V
- net +12V: now also J4.1 (Pin_1), J5.1 (Pin_1); no longer C1.2
- removed net 3V3_EEPROM: J4.2 (Pin_2), R10.1, R12.1, R14.1, R16.2, R3.1, R4.2, U2.8 (VCC)
- net 5V_ALW renamed +5V
- net GPIO0: no longer names the net of J1.PG1 (GPIO0_EC)
- net GPIO1: no longer names the net of J1.PH1 (GPIO1_EC)
- new net: R18.1, SW1.5 (B)
- new net: R19.1, SW2.5 (B)
- new net CLKE_BIAS: R1.2, R2.2, U1.2 (-), U1.6 (-)
- no-connect marks 0 -> 56
Other:
- note added: "CLK enable"
- note added: "Chooses between the global RST or independent ones. This is needed when two 4I devices are connected."
- note added: "EEPROM"
- note added: "FANs"
- note added: "FXBeam"
- note added: "Internal USB"
- note added: "Mounting"
- note added: "NPIO"
- note added: "RST"
- note added: "Since there is no request clock on the connector, it needs to be generated from the presence or not of a device. It can be forced ON with the DIP switches as some docks might not have the pull down for the detection."
- note added: "USB"
- note removed: "Pull-up to 3.3V"
- moved on the sheet: C2, H1, H2, H3, H4, J1A, J1B, J2, J3, R10, R11, R12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

Commit message: updated FXBeam with correct input / outputs for ERC
Updated the FXBeam symbol to have the correct input / outputs instead of unspecified for a bunch of them.
It now passes ERC without a single error / warning.
Parts:
- renumbered SW2 to SW1, SW3 to SW2
Connections:
- net CLK_AUTO_EN1: now also SW1.3 (C); no longer SW1.6 (C)
- net GND: now also J3.SH (Shield), SW1.1 (A); no longer J3.5 (Shield), SW1.4 (A)
- net at R18.1: now also SW1.2 (B); no longer SW1.5 (B)
Other:
- moved on the sheet: H1, H2, H3, H4

Commit message: added ESD diodes
Added the ESD diodes for the external connector.
All the same, as it doesn't really make sense for such a low volume board to optimise costs with different low speed ones for the 3V3 signals.
Technically it means that they are protected for 3.6V instead of 3.3V, but it should be fine.
Parts:
- added D1, D10, D11, D12, D13, D14, D15, D16, D17, D18, D19, D2, D20, D21, D22, D23, D24, D25, D26, D27, D28, D29, D3, D30, D31, D32, D33, D34, D35, D36, D37, D38, D39, D4, D40, D5, D6, D7, D8, D9: TPD1E01B04, Package_SON:Texas_DPY0002A_0.6x1mm_P0.65mm, symbol Device:D_Small
- R19: now not fitted
- U1: footprint Package_DIP:DIP-14_W7.62mm -> Package_SO:TSSOP-8_4.4x3mm_P0.65mm
Connections:
- net CPRSNTA: now also D26.1 (K)
- net CPRSNTB: now also D36.1 (K)
- net GND: now also D1.2 (A), D10.2 (A), D11.2 (A), D12.2 (A), D13.2 (A), D14.2 (A), D15.2 (A), D16.2 (A), D17.2 (A), D18.2 (A), D19.2 (A), D2.2 (A), D20.2 (A), D21.2 (A), D22.2 (A), D23.2 (A), D24.2 (A), D25.2 (A), D26.2 (A), D27.2 (A), D28.2 (A), D29.2 (A), D3.2 (A), D30.2 (A), D31.2 (A), D32.2 (A), D33.2 (A), D34.2 (A), D35.2 (A), D36.2 (A), D37.2 (A), D38.2 (A), D39.2 (A), D4.2 (A), D40.2 (A), D5.2 (A), D6.2 (A), D7.2 (A), D8.2 (A), D9.2 (A)
- net PERSTA: now also D25.1 (K)
- net PERSTB: now also D35.1 (K)
- net REFCLKA+: now also D5.1 (K)
- net REFCLKA-: now also D6.1 (K)
- net REFCLKB+: now also D16.1 (K)
- net REFCLKB-: now also D15.1 (K)
- net RX0+: now also D2.1 (K)
- net RX0-: now also D1.1 (K)
- net RX1+: now also D3.1 (K)
- net RX1-: now also D4.1 (K)
- net RX2+: now also D7.1 (K)
- net RX2-: now also D8.1 (K)
- net RX3+: now also D10.1 (K)
- net RX3-: now also D9.1 (K)
- net RX4+: now also D12.1 (K)
- net RX4-: now also D11.1 (K)
- net RX5+: now also D13.1 (K)
- net RX5-: now also D14.1 (K)
- net RX6+: now also D17.1 (K)
- net RX6-: now also D18.1 (K)
- net RX7+: now also D19.1 (K)
- net RX7-: now also D20.1 (K)
- net TX0+: now also D22.1 (K)
- net TX0-: now also D21.1 (K)
- net TX1+: now also D24.1 (K)
- net TX1-: now also D23.1 (K)
- net TX2+: now also D27.1 (K)
- net TX2-: now also D28.1 (K)
- net TX3+: now also D30.1 (K)
- net TX3-: now also D29.1 (K)
- net TX4+: now also D32.1 (K)
- net TX4-: now also D31.1 (K)
- net TX5+: now also D33.1 (K)
- net TX5-: now also D34.1 (K)
- net TX6+: now also D38.1 (K)
- net TX6-: now also D37.1 (K)
- net TX7+: now also D39.1 (K)
- net TX7-: now also D40.1 (K)
Other:
- note added: "All the same diodes, as putting different ones doesn't make sense BOM wise. It should be fine for all signals as it protects +-3.6V (so okay for the 3V3 signals) It's not the "best" (I.E. specific protection for each signal) but better than nothing."
- note added: "ESD protection"

Commit message: updated PCB shape to be smaller than 10x10cm
All the important things should still be in their right place. The outline is well defined.
One of the mounting hole had to be truncated, may need a small spacer to screw flat.
Parts:
- removed H3, H4: MountingHole_Pad, Expansion_Bay:MountingHole_6.2mm_EasySolder_Cut, symbol Mechanical:MountingHole_Pad
Changed lines of the file:
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@@
 	)
 	(junction
-		(at 375.92 36.83)
-		(diameter 0)
-		(color 0 0 0 0)
-	)
-	(junction
 		(at 378.46 189.23)
 		(diameter 0)
@@
 	)
 	(junction
-		(at 381 36.83)
-		(diameter 0)
-		(color 0 0 0 0)
-	)
-	(junction
 		(at 45.72 255.27)
 		(diameter 0)
@@
 	(wire
 		(pts
-			(xy 381 34.29) (xy 381 36.83)
-		)
-		(stroke
-			(width 0)
-			(type default)
-		)
-	)
-	(wire
-		(pts
 			(xy 182.88 53.34) (xy 195.58 53.34)
 		)
@@
 	(wire
 		(pts
-			(xy 375.92 36.83) (xy 381 36.83)
-		)
-		(stroke
-			(width 0)
-			(type default)
-		)
-	)
-	(wire
-		(pts
 			(xy 120.65 251.46) (xy 120.65 248.92)
 		)
@@
 	(wire
 		(pts
-			(xy 381 36.83) (xy 386.08 36.83)
-		)
-		(stroke
-			(width 0)
-			(type default)
-		)
-	)
-	(wire
-		(pts
 			(xy 111.76 66.04) (xy 102.87 66.04)
 		)
@@
 	(wire
 		(pts
-			(xy 386.08 34.29) (xy 386.08 36.83)
-		)
-		(stroke
-			(width 0)
-			(type default)
-		)
-	)
-	(wire
-		(pts
 			(xy 25.4 123.19) (xy 35.56 123.19)
 		)
@@
 	)
 	(symbol
-		(lib_id "Mechanical:MountingHole_Pad")
-		(at 381 31.75 0)
-		(unit 1)
-		(body_style 1)
-		(exclude_from_sim no)
-		(in_bom no)
-		(on_board yes)
-		(in_pos_files yes)
-		(dnp no)
-		(property "Reference" "H3"
-			(at 379.73 27.432 0)
-			(show_name no)
-			(do_not_autoplace no)
-			(effects
-				(font
-					(size 1.27 1.27)
-				)
-				(justify left)
-			)
-		)
-		(property "Value" "MountingHole_Pad"
-			(at 383.54 31.7499 0)
-			(hide yes)
-			(show_name no)
-			(do_not_autoplace no)
-			(effects
-				(font
-					(size 1.27 1.27)
-				)
-				(justify left)
-			)
-		)
-		(property "Footprint" "Expansion_Bay:MountingHole_6.2mm_EasySolder_Cut"
-			(at 381 31.75 0)
-			(hide yes)
-			(show_name no)
-			(do_not_autoplace no)
-			(effects
-				(font
-					(size 1.27 1.27)
-				)
-			)
-		)
-		(property "Datasheet" ""
-			(at 381 31.75 0)
-			(hide yes)
-			(show_name no)
-			(do_not_autoplace no)
-			(effects
-				(font
-					(size 1.27 1.27)
-				)
-			)
-		)
-		(property "Description" "Mounting Hole with connection"
-			(at 381 31.75 0)
-			(hide yes)
-			(show_name no)
-			(do_not_autoplace no)
-			(effects
-				(font
-					(size 1.27 1.27)
-				)
-			)
-		)
-		(pin "1"
-		)
-		(instances
-			(project "fw16_oculink8i"
-				(path "/50f5fd03-67f8-43d1-8bfe-dca2cf908bf0"
-					(reference "H3")
-					(unit 1)
-				)
-			)
-		)
-	)
-	(symbol
 		(lib_id "power:+12V")
 		(at 342.9 30.48 0)
@@
 					(unit 1)
 				)
-			)
-		)
-	)
-	(symbol
-		(lib_id "Mechanical:MountingHole_Pad")
-		(at 386.08 31.75 0)
-		(unit 1)
-		(body_style 1)
-		(exclude_from_sim no)
-		(in_bom no)
-		(on_board yes)
-		(in_pos_files yes)
-		(dnp no)
-		(property "Reference" "H4"
-			(at 384.81 27.686 0)
-			(show_name no)
-			(do_not_autoplace no)
-			(effects
-				(font
-					(size 1.27 1.27)
-				)
-				(justify left)
-			)
-		)
-		(property "Value" "MountingHole_Pad"
-			(at 388.62 31.7499 0)
-			(hide yes)
-			(show_name no)
-			(do_not_autoplace no)
-			(effects
-				(font
-					(size 1.27 1.27)
-				)
-				(justify left)
-			)
-		)
-		(property "Footprint" "Expansion_Bay:MountingHole_6.2mm_EasySolder_Cut"
-			(at 386.08 31.75 0)
-			(hide yes)
-			(show_name no)
-			(do_not_autoplace no)
-			(effects
-				(font
-					(size 1.27 1.27)
-				)
-			)
-		)
-		(property "Datasheet" ""
-			(at 386.08 31.75 0)
-			(hide yes)
-			(show_name no)
-			(do_not_autoplace no)
-			(effects
-				(font
-					(size 1.27 1.27)
-				)
-			)
-		)
-		(property "Description" "Mounting Hole with connection"
-			(at 386.08 31.75 0)
-			(hide yes)
-			(show_name no)
-			(do_not_autoplace no)
-			(effects
-				(font
-					(size 1.27 1.27)
-				)
-			)
-		)
-		(pin "1"
-		)
-		(instances
-			(project "fw16_oculink8i"
-				(path "/50f5fd03-67f8-43d1-8bfe-dca2cf908bf0"
-					(reference "H4")
-					(unit 1)
-				)

Commit message: routed the boards - passes ERC
Routing done - still need to take care of the silkscreen
Connections:
- net REFCLKB+: now also J2.A32; no longer J2.A33
- net REFCLKB-: now also J2.A33; no longer J2.A32
- net RX2+: now also J1.SD6 (PEX_RX2N); no longer J1.SE6 (PEX_RX2P)
- net RX2-: now also J1.SE6 (PEX_RX2P); no longer J1.SD6 (PEX_RX2N)
- net TX4+: now also J1.SL3 (PEX_TX4N); no longer J1.SK3 (PEX_TX4P)
- net TX4-: now also J1.SK3 (PEX_TX4P); no longer J1.SL3 (PEX_TX4N)
Changed lines of the file:
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@@
 	)
 	(label "TX4-"
-		(at 102.87 66.04 0)
+		(at 102.87 63.5 0)
 		(effects
 			(font
@@
 	)
 	(label "TX4+"
-		(at 102.87 63.5 0)
+		(at 102.87 66.04 0)
 		(effects
 			(font
@@
 	)
 	(label "REFCLKB+"
-		(at 185.42 119.38 0)
+		(at 185.42 116.84 0)
 		(effects
 			(font
@@
 	)
 	(label "RX2-"
-		(at 158.75 55.88 180)
+		(at 158.75 53.34 180)
 		(effects
 			(font
@@
 	)
 	(label "REFCLKB-"
-		(at 185.42 116.84 0)
+		(at 185.42 119.38 0)
 		(effects
 			(font
@@
 	)
 	(label "RX2+"
-		(at 158.75 53.34 180)
-		(effects
-			(font
+		(at 158.75 55.88 180)
+		(effects
+			(font

Commit message: updated footprint for comparator for SOIC-8
JLCPCB has it as a standard component instead of extended, so 3 bucks cheaper (yay)
Parts:
- U1: footprint Package_SO:TSSOP-8_4.4x3mm_P0.65mm -> Package_SO:SOIC-8_3.9x4.9mm_P1.27mm
Changed lines of the file:
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@@
 			)
 		)
-		(property "Footprint" "Package_SO:TSSOP-8_4.4x3mm_P0.65mm"
+		(property "Footprint" "Package_SO:SOIC-8_3.9x4.9mm_P1.27mm"
 			(at 40.64 255.27 0)
 			(hide yes)
@@
 			)
 		)
-		(property "Footprint" "Package_SO:TSSOP-8_4.4x3mm_P0.65mm"
+		(property "Footprint" "Package_SO:SOIC-8_3.9x4.9mm_P1.27mm"
 			(at 83.82 267.97 0)
 			(hide yes)
@@
 			)
 		)
-		(property "Footprint" "Package_SO:TSSOP-8_4.4x3mm_P0.65mm"
+		(property "Footprint" "Package_SO:SOIC-8_3.9x4.9mm_P1.27mm"
 			(at 83.82 247.65 0)
 			(hide yes)
